File: Hardware/Motor Drivers.sch (KiCad schematic (older format))
At the start: 22 parts

Commit message: Motor driver and power management subsheet converted to blocks
Parts:
- removed C?: 10uF, Capacitor_SMD:C_2220_5650Metric, symbol Device:C_Small
- removed C?: 1uF, Resistor_SMD:R_0603_1608Metric, symbol Device:C_Small
- removed C?: 100nF, Resistor_SMD:R_0603_1608Metric, symbol Device:C_Small
- removed C?: 22nF, Resistor_SMD:R_0603_1608Metric, symbol Device:C_Small
- removed R?: 5.5k, Resistor_SMD:R_0603_1608Metric, symbol Device:R_Small_US
- removed R?: 16k, Resistor_SMD:R_0603_1608Metric, symbol Device:R_Small_US
- removed R?: 50k, Resistor_SMD:R_0603_1608Metric, symbol Device:R_Small_US
- removed R?: 10k, Resistor_SMD:R_0603_1608Metric, symbol Device:R_Small_US
- removed TP? (x2): M+, TestPoint:TestPoint_Keystone_5000-5004_Miniature, symbol Connector:TestPoint
- removed TP? (x2): M-, TestPoint:TestPoint_Keystone_5000-5004_Miniature, symbol Connector:TestPoint
- removed U?: DRV8874, Package_SO:HTSSOP-16-1EP_4.4x5mm_P0.65mm_EP3.4x5mm_Mask3x3mm_ThermalVias, symbol Driver_Motor:DRV8874
Other:
- moved on the sheet: C?, R?, U?
