File: Hardware/Peripherals.sch (KiCad schematic (older format))
At the start: 0 parts

Commit message: Motor driver and power management subsheet converted to blocks
Parts:
- added U3: BME280, Package_LGA:Bosch_LGA-8_2.5x2.5mm_P0.65mm_ClockwisePinNumbering, symbol Sensor:BME280
Changed lines of the file:
@@
 $Descr A4 11693 8268
 encoding utf-8
-Sheet 1 5
+Sheet 5 6
 Title ""
 Date ""
@@
 Comment4 ""
 $EndDescr
+$Comp
+L Sensor:BME280 U3
+U 1 1 5FEDA4A0
+P 5900 3900
+F 0 "U3" H 5471 3946 50  0000 R CNN
+F 1 "BME280" H 5471 3855 50  0000 R CNN
+F 2 "Package_LGA:Bosch_LGA-8_2.5x2.5mm_P0.65mm_ClockwisePinNumbering" H 7400 3450 50  0001 C CNN
+F 3 "https://ae-bst.resource.bosch.com/media/_tech/media/datasheets/BST-BME280-DS002.pdf" H 5900 3700 50  0001 C CNN
+	1    5900 3900
+	1    0    0    -1
+$EndComp
 $EndSCHEMATC
