File: Hardware/Peripherals.sch (KiCad schematic (older format))
At the start: 1 part, among them U3 BME280

Commit message: Readme updated
Parts:
- renumbered U3 to U4
Changed lines of the file:
@@
 $EndDescr
 $Comp
-L Sensor:BME280 U3
+L Sensor:BME280 U4
 U 1 1 5FEDA4A0
 P 5900 3900
-F 0 "U3" H 5471 3946 50  0000 R CNN
+F 0 "U4" H 5471 3946 50  0000 R CNN
 F 1 "BME280" H 5471 3855 50  0000 R CNN
 F 2 "Package_LGA:Bosch_LGA-8_2.5x2.5mm_P0.65mm_ClockwisePinNumbering" H 7400 3450 50  0001 C CNN
