File: Hardware/MCU.sch (KiCad schematic (older format))
At the start: 11 parts

Commit message: Motor driver and power management subsheet converted to blocks
Parts:
- gave numbers to parts that had none: 11
Changed lines of the file:
@@
 $Descr A4 11693 8268
 encoding utf-8
-Sheet 2 5
+Sheet 2 6
 Title ""
 Date ""
@@
 AR Path="/5EA2026E/5FF09BD0" Ref="#PWR?"  Part="1"
 AR Path="/5FF09BD0" Ref="#PWR?"  Part="1"
-F 0 "#PWR?" H 4050 2400 50  0001 C CNN
+AR Path="/5FEFFC20/5FF09BD0" Ref="#PWR02"  Part="1"
+F 0 "#PWR02" H 4050 2400 50  0001 C CNN
 F 1 "+3.3V" H 4065 2723 50  0000 C CNN
 F 2 "" H 4050 2550 50  0001 C CNN
@@
 AR Path="/5EA2026E/5FF09BD7" Ref="C?"  Part="1"
 AR Path="/5FF09BD7" Ref="C?"  Part="1"
-F 0 "C?" V 4050 4800 50  0000 C CNN
+AR Path="/5FEFFC20/5FF09BD7" Ref="C3"  Part="1"
+F 0 "C3" V 4050 4800 50  0000 C CNN
 F 1 "100nF" V 4050 5050 50  0000 C CNN
 F 2 "Capacitor_SMD:C_0805_2012Metric" H 4000 4900 50  0001 C CNN
@@
 BOOT
 $Comp
-L RF_Module:ESP32-WROOM-32U U?
+L RF_Module:ESP32-WROOM-32U U1
 U 1 1 5FF09BE4
 P 5500 3700
-F 0 "U?" H 5950 5200 50  0000 C CNN
+F 0 "U1" H 5950 5200 50  0000 C CNN
 F 1 "ESP32-WROOM-32U" H 5950 5100 50  0000 C CNN
 F 2 "RF_Module:ESP32-WROOM-32U" H 5500 2200 50  0001 C CNN
@@
 BOOT
 $Comp
-L power:GND #PWR?
+L power:GND #PWR011
 U 1 1 5FF09BF4
 P 5500 5100
-F 0 "#PWR?" H 5500 4850 50  0001 C CNN
+F 0 "#PWR011" H 5500 4850 50  0001 C CNN
 F 1 "GND" H 5505 4927 50  0000 C CNN
 F 2 "" H 5500 5100 50  0001 C CNN
@@
 AR Path="/5EA2026E/5FF09C02" Ref="C?"  Part="1"
 AR Path="/5FF09C02" Ref="C?"  Part="1"
-F 0 "C?" V 4050 3800 50  0000 C CNN
+AR Path="/5FEFFC20/5FF09C02" Ref="C2"  Part="1"
+F 0 "C2" V 4050 3800 50  0000 C CNN
 F 1 "100nF" V 4050 4050 50  0000 C CNN
 F 2 "Capacitor_SMD:C_0805_2012Metric" H 4000 3900 50  0001 C CNN
@@
 AR Path="/5EA2026E/5FF09C08" Ref="#PWR?"  Part="1"
 AR Path="/5FF09C08" Ref="#PWR?"  Part="1"
-F 0 "#PWR?" H 4050 2500 50  0001 C CNN
+AR Path="/5FEFFC20/5FF09C08" Ref="#PWR03"  Part="1"
+F 0 "#PWR03" H 4050 2500 50  0001 C CNN
 F 1 "GND" H 4055 2577 50  0000 C CNN
 F 2 "" H 4050 2750 50  0001 C CNN
@@
 AR Path="/5EA2026E/5FF09C0E" Ref="C?"  Part="1"
 AR Path="/5FF09C0E" Ref="C?"  Part="1"
-F 0 "C?" H 4142 2696 50  0000 L CNN
+AR Path="/5FEFFC20/5FF09C0E" Ref="C1"  Part="1"
+F 0 "C1" H 4142 2696 50  0000 L CNN
 F 1 "100nF" H 4142 2605 50  0000 L CNN
 F 2 "Capacitor_SMD:C_0805_2012Metric" H 4050 2650 50  0001 C CNN
@@
 AR Path="/5EA2026E/5FF09C14" Ref="#PWR?"  Part="1"
 AR Path="/5FF09C14" Ref="#PWR?"  Part="1"
-F 0 "#PWR?" H 4250 3200 50  0001 C CNN
+AR Path="/5FEFFC20/5FF09C14" Ref="#PWR04"  Part="1"
+F 0 "#PWR04" H 4250 3200 50  0001 C CNN
 F 1 "+3.3V" H 4265 3523 50  0000 C CNN
 F 2 "" H 4250 3350 50  0001 C CNN
@@
 AR Path="/5EA2026E/5FF09C1A" Ref="R?"  Part="1"
 AR Path="/5FF09C1A" Ref="R?"  Part="1"
-F 0 "R?" H 4318 3496 50  0000 L CNN
+AR Path="/5FEFFC20/5FF09C1A" Ref="R1"  Part="1"
+F 0 "R1" H 4318 3496 50  0000 L CNN
 F 1 "10k" H 4318 3405 50  0000 L CNN
 F 2 "Resistor_SMD:R_0805_2012Metric" H 4250 3450 50  0001 C CNN
@@
 	4250 3550 4250 3600
 $Comp
-L power:GND #PWR?
+L power:GND #PWR06
 U 1 1 5FF09C21
 P 3700 3750
-F 0 "#PWR?" H 3700 3500 50  0001 C CNN
+F 0 "#PWR06" H 3700 3500 50  0001 C CNN
 F 1 "GND" V 3705 3622 50  0000 R CNN
 F 2 "" H 3700 3750 50  0001 C CNN
@@
 	3750 3750 3750 3600
 $Comp
-L power:GND #PWR?
+L power:GND #PWR010
 U 1 1 5FF09C2A
 P 3700 4750
-F 0 "#PWR?" H 3700 4500 50  0001 C CNN
+F 0 "#PWR010" H 3700 4500 50  0001 C CNN
 F 1 "GND" V 3705 4622 50  0000 R CNN
 F 2 "" H 3700 4750 50  0001 C CNN
@@
 	3750 4750 3750 4600
 $Comp
-L power:+3.3V #PWR?
+L power:+3.3V #PWR01
 U 1 1 5FF09C33
 P 5500 2300
-F 0 "#PWR?" H 5500 2150 50  0001 C CNN
+F 0 "#PWR01" H 5500 2150 50  0001 C CNN
 F 1 "+3.3V" H 5515 2473 50  0000 C CNN
 F 2 "" H 5500 2300 50  0001 C CNN
@@
 $EndComp
 $Comp
-L Device:R_Small_US R?
+L Device:R_Small_US R3
 U 1 1 5FF09C39
 P 7000 4350
-F 0 "R?" H 7068 4396 50  0000 L CNN
+F 0 "R3" H 7068 4396 50  0000 L CNN
 F 1 "4.7k" H 7068 4305 50  0000 L CNN
 F 2 "Resistor_SMD:R_0603_1608Metric" H 7000 4350 50  0001 C CNN
@@
 $EndComp
 $Comp
-L Device:R_Small_US R?
+L Device:R_Small_US R2
 U 1 1 5FF09C3F
 P 6650 4350
-F 0 "R?" H 6718 4396 50  0000 L CNN
+F 0 "R2" H 6718 4396 50  0000 L CNN
 F 1 "4.7k" H 6718 4305 50  0000 L CNN
 F 2 "Resistor_SMD:R_0603_1608Metric" H 6650 4350 50  0001 C CNN
@@
 SCL
 $Comp
-L power:+3.3V #PWR?
+L power:+3.3V #PWR07
 U 1 1 5FF09C47
 P 6650 4250
-F 0 "#PWR?" H 6650 4100 50  0001 C CNN
+F 0 "#PWR07" H 6650 4100 50  0001 C CNN
 F 1 "+3.3V" H 6665 4423 50  0000 C CNN
 F 2 "" H 6650 4250 50  0001 C CNN
@@
 $EndComp
 $Comp
-L power:+3.3V #PWR?
+L power:+3.3V #PWR08
 U 1 1 5FF09C4D
 P 7000 4250
-F 0 "#PWR?" H 7000 4100 50  0001 C CNN
+F 0 "#PWR08" H 7000 4100 50  0001 C CNN
 F 1 "+3.3V" H 7015 4423 50  0000 C CNN
 F 2 "" H 7000 4250 50  0001 C CNN
@@
 NoConn ~ 6100 4600
 $Comp
-L Switch:SW_Push SW?
+L Switch:SW_Push SW1
 U 1 1 5FF09C67
 P 4000 3600
-F 0 "SW?" H 4000 3885 50  0000 C CNN
+F 0 "SW1" H 4000 3885 50  0000 C CNN
 F 1 "SW_Push" H 4000 3794 50  0001 C CNN
 F 2 "Button_Switch_SMD:SW_SPST_CK_RS282G05A3" H 4000 3800 50  0001 C CNN
@@
 	4100 3900 4250 3900
 $Comp
-L Switch:SW_Push SW?
+L Switch:SW_Push SW2
 U 1 1 5FF09C70
 P 4000 4600
-F 0 "SW?" H 4000 4885 50  0000 C CNN
+F 0 "SW2" H 4000 4885 50  0000 C CNN
 F 1 "SW_Push" H 4000 4794 50  0001 C CNN
 F 2 "Button_Switch_SMD:SW_SPST_CK_RS282G05A3" H 4000 4800 50  0001 C CNN
@@
 AR Path="/5EA2026E/5FF09C78" Ref="#PWR?"  Part="1"
 AR Path="/5FF09C78" Ref="#PWR?"  Part="1"
-F 0 "#PWR?" H 4250 4200 50  0001 C CNN
+AR Path="/5FEFFC20/5FF09C78" Ref="#PWR09"  Part="1"
+F 0 "#PWR09" H 4250 4200 50  0001 C CNN
 F 1 "+3.3V" H 4265 4523 50  0000 C CNN
 F 2 "" H 4250 4350 50  0001 C CNN
@@
 AR Path="/5EA2026E/5FF09C7E" Ref="R?"  Part="1"
 AR Path="/5FF09C7E" Ref="R?"  Part="1"
-F 0 "R?" H 4318 4496 50  0000 L CNN
+AR Path="/5FEFFC20/5FF09C7E" Ref="R4"  Part="1"
+F 0 "R4" H 4318 4496 50  0000 L CNN
 F 1 "10k" H 4318 4405 50  0000 L CNN
 F 2 "Resistor_SMD:R_0805_2012Metric" H 4250 4450 50  0001 C CNN
@@
 	4250 4550 4250 4600
 $Comp
-L Connector_Generic:Conn_01x03 J?
+L Connector_Generic:Conn_01x03 J1
 U 1 1 5FF09C86
 P 6950 3250
-F 0 "J?" H 7030 3337 50  0000 L CNN
+F 0 "J1" H 7030 3337 50  0000 L CNN
 F 1 "HDR" H 7030 3246 50  0000 L CNN
 F 2 "" H 6950 3250 50  0001 C CNN
@@
 TX
 $Comp
-L power:GND #PWR?
+L power:GND #PWR05
 U 1 1 5FF09C90
 P 6750 3350
-F 0 "#PWR?" H 6750 3100 50  0001 C CNN
+F 0 "#PWR05" H 6750 3100 50  0001 C CNN
 F 1 "GND" V 6755 3222 50  0000 R CNN
 F 2 "" H 6750 3350 50  0001 C CNN

Commit message: Signed-off-by: Usman Mehmood <usmanmehmood55@gmail.com>
Connections:
- net labels added: CHG, FAULT_L, FAULT_R, FSYNC, INT, IR_L, IR_R, PG, PH_L, PH_R, PWM_L, PWM_R, SLEEP_L, SLEEP_R, iPROPI_L, iPROPI_R
- no-connect marks 27 -> 11
Other:
- note removed: "To be replaced by ESP32 Cam"
- moved on the sheet: C1, C2, C3, J1, R1, R2, R3, R4, SW1, SW2

Commit message: Replaced ESP-WROOM-32D with ESP32-CAM
Parts:
- removed U1: ESP32-WROOM-32U, RF_Module:ESP32-WROOM-32U, symbol RF_Module:ESP32-WROOM-32U
- added U?: ESP32-CAM, symbol RF_Module:ESP32-CAM
- renumbered C2 to C10, C3 to C11, C1 to C9, R1 to R13, R4 to R14, R2 to R15, R3 to R16
Changed lines of the file:
@@
 AR Path="/5EA2026E/5FF09BD0" Ref="#PWR?"  Part="1"
 AR Path="/5FF09BD0" Ref="#PWR?"  Part="1"
-AR Path="/5FEFFC20/5FF09BD0" Ref="#PWR05"  Part="1"
-F 0 "#PWR05" H 3750 2400 50  0001 C CNN
+AR Path="/5FEFFC20/5FF09BD0" Ref="#PWR035"  Part="1"
+F 0 "#PWR035" H 3750 2400 50  0001 C CNN
 F 1 "+3.3V" H 3765 2723 50  0000 C CNN
 F 2 "" H 3750 2550 50  0001 C CNN
@@
 AR Path="/5EA2026E/5FF09BD7" Ref="C?"  Part="1"
 AR Path="/5FF09BD7" Ref="C?"  Part="1"
-AR Path="/5FEFFC20/5FF09BD7" Ref="C3"  Part="1"
-F 0 "C3" V 3750 4800 50  0000 C CNN
+AR Path="/5FEFFC20/5FF09BD7" Ref="C11"  Part="1"
+F 0 "C11" V 3750 4800 50  0000 C CNN
 F 1 "100nF" V 3750 5050 50  0000 C CNN
 F 2 "Capacitor_SMD:C_0805_2012Metric" H 3700 4900 50  0001 C CNN
@@
 Text GLabel 4000 4600 2    50   Output ~ 0
 BOOT
-$Comp
-L RF_Module:ESP32-WROOM-32U U1
-U 1 1 5FF09BE4
-P 6000 3800
-F 0 "U1" H 6450 5300 50  0000 C CNN
-F 1 "ESP32-WROOM-32U" H 6450 5200 50  0000 C CNN
-F 2 "RF_Module:ESP32-WROOM-32U" H 6000 2300 50  0001 C CNN
-F 3 "https://www.espressif.com/sites/default/files/documentation/esp32-wroom-32d_esp32-wroom-32u_datasheet_en.pdf" H 5700 3850 50  0001 C CNN
-	1    6000 3800
-	1    0    0    -1
-$EndComp
 NoConn ~ 5400 3800
 NoConn ~ 5400 3900
@@
 BOOT
 $Comp
-L power:GND #PWR014
+L power:GND #PWR044
 U 1 1 5FF09BF4
 P 6000 5200
-F 0 "#PWR014" H 6000 4950 50  0001 C CNN
+F 0 "#PWR044" H 6000 4950 50  0001 C CNN
 F 1 "GND" H 6005 5027 50  0000 C CNN
 F 2 "" H 6000 5200 50  0001 C CNN
@@
 AR Path="/5EA2026E/5FF09C02" Ref="C?"  Part="1"
 AR Path="/5FF09C02" Ref="C?"  Part="1"
-AR Path="/5FEFFC20/5FF09C02" Ref="C2"  Part="1"
-F 0 "C2" V 3750 3800 50  0000 C CNN
+AR Path="/5FEFFC20/5FF09C02" Ref="C10"  Part="1"
+F 0 "C10" V 3750 3800 50  0000 C CNN
 F 1 "100nF" V 3750 4050 50  0000 C CNN
 F 2 "Capacitor_SMD:C_0805_2012Metric" H 3700 3900 50  0001 C CNN
@@
 AR Path="/5EA2026E/5FF09C08" Ref="#PWR?"  Part="1"
 AR Path="/5FF09C08" Ref="#PWR?"  Part="1"
-AR Path="/5FEFFC20/5FF09C08" Ref="#PWR06"  Part="1"
-F 0 "#PWR06" H 3750 2500 50  0001 C CNN
+AR Path="/5FEFFC20/5FF09C08" Ref="#PWR036"  Part="1"
+F 0 "#PWR036" H 3750 2500 50  0001 C CNN
 F 1 "GND" H 3755 2577 50  0000 C CNN
 F 2 "" H 3750 2750 50  0001 C CNN
@@
 AR Path="/5EA2026E/5FF09C0E" Ref="C?"  Part="1"
 AR Path="/5FF09C0E" Ref="C?"  Part="1"
-AR Path="/5FEFFC20/5FF09C0E" Ref="C1"  Part="1"
-F 0 "C1" H 3842 2696 50  0000 L CNN
+AR Path="/5FEFFC20/5FF09C0E" Ref="C9"  Part="1"
+F 0 "C9" H 3842 2696 50  0000 L CNN
 F 1 "100nF" H 3842 2605 50  0000 L CNN
 F 2 "Capacitor_SMD:C_0805_2012Metric" H 3750 2650 50  0001 C CNN
@@
 AR Path="/5EA2026E/5FF09C14" Ref="#PWR?"  Part="1"
 AR Path="/5FF09C14" Ref="#PWR?"  Part="1"
-AR Path="/5FEFFC20/5FF09C14" Ref="#PWR07"  Part="1"
-F 0 "#PWR07" H 3950 3200 50  0001 C CNN
+AR Path="/5FEFFC20/5FF09C14" Ref="#PWR038"  Part="1"
+F 0 "#PWR038" H 3950 3200 50  0001 C CNN
 F 1 "+3.3V" H 3965 3523 50  0000 C CNN
 F 2 "" H 3950 3350 50  0001 C CNN
@@
 AR Path="/5EA2026E/5FF09C1A" Ref="R?"  Part="1"
 AR Path="/5FF09C1A" Ref="R?"  Part="1"
-AR Path="/5FEFFC20/5FF09C1A" Ref="R1"  Part="1"
-F 0 "R1" H 4018 3496 50  0000 L CNN
+AR Path="/5FEFFC20/5FF09C1A" Ref="R13"  Part="1"
+F 0 "R13" H 4018 3496 50  0000 L CNN
 F 1 "10k" H 4018 3405 50  0000 L CNN
 F 2 "Resistor_SMD:R_0805_2012Metric" H 3950 3450 50  0001 C CNN
@@
 	3950 3550 3950 3600
 $Comp
-L power:GND #PWR09
+L power:GND #PWR039
 U 1 1 5FF09C21
 P 3400 3750
-F 0 "#PWR09" H 3400 3500 50  0001 C CNN
+F 0 "#PWR039" H 3400 3500 50  0001 C CNN
 F 1 "GND" V 3405 3622 50  0000 R CNN
 F 2 "" H 3400 3750 50  0001 C CNN
@@
 	3450 3750 3450 3600
 $Comp
-L power:GND #PWR013
+L power:GND #PWR043
 U 1 1 5FF09C2A
 P 3400 4750
-F 0 "#PWR013" H 3400 4500 50  0001 C CNN
+F 0 "#PWR043" H 3400 4500 50  0001 C CNN
 F 1 "GND" V 3405 4622 50  0000 R CNN
 F 2 "" H 3400 4750 50  0001 C CNN
@@
 	3450 4750 3450 4600
 $Comp
-L power:+3.3V #PWR04
+L power:+3.3V #PWR034
 U 1 1 5FF09C33
 P 6000 2400
-F 0 "#PWR04" H 6000 2250 50  0001 C CNN
+F 0 "#PWR034" H 6000 2250 50  0001 C CNN
 F 1 "+3.3V" H 6015 2573 50  0000 C CNN
 F 2 "" H 6000 2400 50  0001 C CNN
@@
 $EndComp
 $Comp
-L Device:R_Small_US R3
+L Device:R_Small_US R16
 U 1 1 5FF09C39
 P 8600 4650
-F 0 "R3" H 8668 4696 50  0000 L CNN
+F 0 "R16" H 8668 4696 50  0000 L CNN
 F 1 "4.7k" H 8668 4605 50  0000 L CNN
 F 2 "Resistor_SMD:R_0603_1608Metric" H 8600 4650 50  0001 C CNN
@@
 $EndComp
 $Comp
-L Device:R_Small_US R2
+L Device:R_Small_US R15
 U 1 1 5FF09C3F
 P 8250 4650
-F 0 "R2" H 8318 4696 50  0000 L CNN
+F 0 "R15" H 8318 4696 50  0000 L CNN
 F 1 "4.7k" H 8318 4605 50  0000 L CNN
 F 2 "Resistor_SMD:R_0603_1608Metric" H 8250 4650 50  0001 C CNN
@@
 SCL
 $Comp
-L power:+3.3V #PWR010
+L power:+3.3V #PWR041
 U 1 1 5FF09C47
 P 8250 4550
-F 0 "#PWR010" H 8250 4400 50  0001 C CNN
+F 0 "#PWR041" H 8250 4400 50  0001 C CNN
 F 1 "+3.3V" H 8265 4723 50  0000 C CNN
 F 2 "" H 8250 4550 50  0001 C CNN
@@
 $EndComp
 $Comp
-L power:+3.3V #PWR011
+L power:+3.3V #PWR042
 U 1 1 5FF09C4D
 P 8600 4550
-F 0 "#PWR011" H 8600 4400 50  0001 C CNN
+F 0 "#PWR042" H 8600 4400 50  0001 C CNN
 F 1 "+3.3V" H 8615 4723 50  0000 C CNN
 F 2 "" H 8600 4550 50  0001 C CNN
@@
 AR Path="/5EA2026E/5FF09C78" Ref="#PWR?"  Part="1"
 AR Path="/5FF09C78" Ref="#PWR?"  Part="1"
-AR Path="/5FEFFC20/5FF09C78" Ref="#PWR012"  Part="1"
-F 0 "#PWR012" H 3950 4200 50  0001 C CNN
+AR Path="/5FEFFC20/5FF09C78" Ref="#PWR040"  Part="1"
+F 0 "#PWR040" H 3950 4200 50  0001 C CNN
 F 1 "+3.3V" H 3965 4523 50  0000 C CNN
 F 2 "" H 3950 4350 50  0001 C CNN
@@
 AR Path="/5EA2026E/5FF09C7E" Ref="R?"  Part="1"
 AR Path="/5FF09C7E" Ref="R?"  Part="1"
-AR Path="/5FEFFC20/5FF09C7E" Ref="R4"  Part="1"
-F 0 "R4" H 4018 4496 50  0000 L CNN
+AR Path="/5FEFFC20/5FF09C7E" Ref="R14"  Part="1"
+F 0 "R14" H 4018 4496 50  0000 L CNN
 F 1 "10k" H 4018 4405 50  0000 L CNN
 F 2 "Resistor_SMD:R_0805_2012Metric" H 3950 4450 50  0001 C CNN
@@
 TX
 $Comp
-L power:GND #PWR08
+L power:GND #PWR037
 U 1 1 5FF09C90
 P 8550 3000
-F 0 "#PWR08" H 8550 2750 50  0001 C CNN
+F 0 "#PWR037" H 8550 2750 50  0001 C CNN
 F 1 "GND" V 8555 2872 50  0000 R CNN
 F 2 "" H 8550 3000 50  0001 C CNN
@@
 NoConn ~ 6600 4800
 NoConn ~ 6600 4900
+$Comp
+L RF_Module:ESP32-CAM U?
+U 1 1 60081D63
+P 6000 3600
+F 0 "U?" H 5672 3671 50  0000 R CNN
+F 1 "ESP32-CAM" H 5672 3580 50  0000 R CNN
+F 2 "" H 6000 5050 50  0001 C CNN
+F 3 "" H 6000 5050 50  0001 C CNN
+	1    6000 3600
+	1    0    0    -1
+$EndComp
 $EndSCHEMATC

Commit message: Signed-off-by: Usman <usmanmehmood55@gmail.com>
Parts:
- removed U?: ESP32-CAM, symbol RF_Module:ESP32-CAM
- added U5: ESP32-WROOM-32D, RF_Module:ESP32-WROOM-32, symbol RF_Module:ESP32-WROOM-32D
- renumbered R13 to R15, R14 to R16, R15 to R17, R16 to R18
Changed lines of the file:
@@
 AR Path="/5EA2026E/5FF09C1A" Ref="R?"  Part="1"
 AR Path="/5FF09C1A" Ref="R?"  Part="1"
-AR Path="/5FEFFC20/5FF09C1A" Ref="R13"  Part="1"
-F 0 "R13" H 4018 3496 50  0000 L CNN
+AR Path="/5FEFFC20/5FF09C1A" Ref="R15"  Part="1"
+F 0 "R15" H 4018 3496 50  0000 L CNN
 F 1 "10k" H 4018 3405 50  0000 L CNN
 F 2 "Resistor_SMD:R_0805_2012Metric" H 3950 3450 50  0001 C CNN
@@
 $EndComp
 $Comp
-L Device:R_Small_US R16
+L Device:R_Small_US R18
 U 1 1 5FF09C39
 P 8600 4650
-F 0 "R16" H 8668 4696 50  0000 L CNN
+F 0 "R18" H 8668 4696 50  0000 L CNN
 F 1 "4.7k" H 8668 4605 50  0000 L CNN
 F 2 "Resistor_SMD:R_0603_1608Metric" H 8600 4650 50  0001 C CNN
@@
 $EndComp
 $Comp
-L Device:R_Small_US R15
+L Device:R_Small_US R17
 U 1 1 5FF09C3F
 P 8250 4650
-F 0 "R15" H 8318 4696 50  0000 L CNN
+F 0 "R17" H 8318 4696 50  0000 L CNN
 F 1 "4.7k" H 8318 4605 50  0000 L CNN
 F 2 "Resistor_SMD:R_0603_1608Metric" H 8250 4650 50  0001 C CNN
@@
 	1    0    0    -1
 $EndComp
-Text GLabel 8600 4750 3    50   UnSpc ~ 0
-SDA
-Text GLabel 8250 4750 3    50   UnSpc ~ 0
-SCL
 $Comp
 L power:+3.3V #PWR041
@@
 AR Path="/5EA2026E/5FF09C7E" Ref="R?"  Part="1"
 AR Path="/5FF09C7E" Ref="R?"  Part="1"
-AR Path="/5FEFFC20/5FF09C7E" Ref="R14"  Part="1"
-F 0 "R14" H 4018 4496 50  0000 L CNN
+AR Path="/5FEFFC20/5FF09C7E" Ref="R16"  Part="1"
+F 0 "R16" H 4018 4496 50  0000 L CNN
 F 1 "10k" H 4018 4405 50  0000 L CNN
 F 2 "Resistor_SMD:R_0805_2012Metric" H 3950 4450 50  0001 C CNN
@@
 NoConn ~ 6600 4900
 $Comp
-L RF_Module:ESP32-CAM U?
-U 1 1 60081D63
-P 6000 3600
-F 0 "U?" H 5672 3671 50  0000 R CNN
-F 1 "ESP32-CAM" H 5672 3580 50  0000 R CNN
-F 2 "" H 6000 5050 50  0001 C CNN
-F 3 "" H 6000 5050 50  0001 C CNN
-	1    6000 3600
-	1    0    0    -1
-$EndComp
+L RF_Module:ESP32-WROOM-32D U5
+U 1 1 607032D0
+P 6000 3800
+F 0 "U5" H 6500 5300 50  0000 C CNN
+F 1 "ESP32-WROOM-32D" H 6500 5200 50  0000 C CNN
+F 2 "RF_Module:ESP32-WROOM-32" H 6000 2300 50  0001 C CNN
+F 3 "https://www.espressif.com/sites/default/files/documentation/esp32-wroom-32d_esp32-wroom-32u_datasheet_en.pdf" H 5700 3850 50  0001 C CNN
+	1    6000 3800
+	1    0    0    -1
+$EndComp
+Text HLabel 8250 4750 3    50   UnSpc ~ 0
+SCL
+Text HLabel 8600 4750 3    50   UnSpc ~ 0
+SDA
 $EndSCHEMATC
