File: Hardware/Motor Driver.sch (KiCad schematic (older format))
At the start: 9 parts, among them U2 DRV8874

Commit message: PCB design started
Parts:
- C1: renamed from C3; symbol Device:C_Small -> Roverette-rescue:C_Small-Device
- C2: renamed from C4; symbol Device:C_Small -> Roverette-rescue:C_Small-Device
- C3: renamed from C1; symbol Device:C_Small -> Roverette-rescue:C_Small-Device
- C4: renamed from C2; symbol Device:C_Small -> Roverette-rescue:C_Small-Device
- R5, R8: symbol Device:R_Small_US -> Roverette-rescue:R_Small_US-Device
- R6: renamed from R7; symbol Device:R_Small_US -> Roverette-rescue:R_Small_US-Device
- R7: renamed from R6; symbol Device:R_Small_US -> Roverette-rescue:R_Small_US-Device
- renumbered U2 to U1
