File: Hardware/USB C.sch (KiCad schematic (older format))
At the start: 2 parts

Commit message: PCB design started
Parts:
- J2: renamed from J?; symbol Connector:USB_C_Receptacle_USB2.0 -> Roverette-rescue:USB_C_Receptacle_USB2.0-Connector
- gave numbers to parts that had none: 1
Changed lines of the file:
@@
 $Descr A4 11693 8268
 encoding utf-8
-Sheet 12 12
+Sheet 11 11
 Title ""
 Date ""
@@
 AR Path="/607FE1AA/6089570F" Ref="U?"  Part="1"
 AR Path="/6089570F" Ref="U?"  Part="1"
-F 0 "U?" H 7230 4121 50  0000 L CNN
+AR Path="/60893A6D/6089570F" Ref="U10"  Part="1"
+F 0 "U10" H 7230 4121 50  0000 L CNN
 F 1 "ESDA6V8AV5" H 7230 4030 50  0000 L CNN
 F 2 "Package_TO_SOT_SMD:SOT-553" H 6650 4550 50  0001 C CNN
@@
 NoConn ~ 7100 4100
 $Comp
-L power:GND #PWR?
+L Roverette-rescue:GND-power #PWR?
 U 1 1 6089571A
 P 6900 4550
 AR Path="/607FE1AA/6089571A" Ref="#PWR?"  Part="1"
 AR Path="/6089571A" Ref="#PWR?"  Part="1"
-F 0 "#PWR?" H 6900 4300 50  0001 C CNN
+AR Path="/60893A6D/6089571A" Ref="#PWR074"  Part="1"
+F 0 "#PWR074" H 6900 4300 50  0001 C CNN
 F 1 "GND" H 6905 4377 50  0000 C CNN
 F 2 "" H 6900 4550 50  0001 C CNN
@@
 $EndComp
 $Comp
-L Connector:USB_C_Receptacle_USB2.0 J?
+L Roverette-rescue:USB_C_Receptacle_USB2.0-Connector J2
 U 1 1 60895724
 P 5850 3850
-F 0 "J?" H 5957 4717 50  0000 C CNN
+F 0 "J2" H 5957 4717 50  0000 C CNN
 F 1 "USB_C_Receptacle" H 5957 4626 50  0000 C CNN
 F 2 "Connector_USB:USB_C_Receptacle_XKB_U262-16XN-4BVC11" H 6000 3850 50  0001 C CNN
@@
 	5850 4800 5850 4750
 $Comp
-L power:GND #PWR?
+L Roverette-rescue:GND-power #PWR?
 U 1 1 6089572D
 P 5700 4850
 AR Path="/607FE1AA/6089572D" Ref="#PWR?"  Part="1"
 AR Path="/6089572D" Ref="#PWR?"  Part="1"
-F 0 "#PWR?" H 5700 4600 50  0001 C CNN
+AR Path="/60893A6D/6089572D" Ref="#PWR073"  Part="1"
+F 0 "#PWR073" H 5700 4600 50  0001 C CNN
 F 1 "GND" H 5705 4677 50  0000 C CNN
 F 2 "" H 5700 4850 50  0001 C CNN
@@
 Wire Wire Line
 	7000 3750 7000 4100
+$Comp
+L Roverette-rescue:PWR_FLAG-power #FLG0103
+U 1 1 6133D762
+P 7000 3200
+F 0 "#FLG0103" H 7000 3275 50  0001 C CNN
+F 1 "PWR_FLAG-power" H 7000 3373 50  0000 C CNN
+F 2 "" H 7000 3200 50  0001 C CNN
+F 3 "" H 7000 3200 50  0001 C CNN
+	1    7000 3200
+	1    0    0    -1
+$EndComp
+Wire Wire Line
+	7000 3200 7000 3250
+Connection ~ 7000 3250
 $EndSCHEMATC
