File: Hardware/USB-TTL.sch (KiCad schematic (older format))
At the start: 9 parts, among them Q1 BSS138, Q2 BSS138, U11 CH340G, Y1 12MHz

Commit message: Schematic and Readme updated
Changed lines of the file:
@@
 $Descr A4 11693 8268
 encoding utf-8
-Sheet 11 11
+Sheet 11 12
 Title "USB Comms"
 Date "2019-01-26"
@@
 Wire Wire Line
 	5850 4300 6450 4300
-Text HLabel 5000 3750 0    50   Input ~ 0
+Text HLabel 5000 3750 0    50   BiDi ~ 0
 D+
-Text HLabel 5000 3850 0    50   Input ~ 0
+Text HLabel 5000 3850 0    50   BiDi ~ 0
 D-
 Text HLabel 5800 3550 2    50   Input ~ 0

Commit message: PCB design started
Parts:
- C26: symbol Device:CP_Small -> Roverette-rescue:CP_Small-Device
- C27: renamed from C29; symbol Device:C_Small -> Roverette-rescue:C_Small-Device
- C28: renamed from C27; symbol Device:C_Small -> Roverette-rescue:C_Small-Device
- C29: renamed from C30; symbol Device:C_Small -> Roverette-rescue:C_Small-Device
- C30: renamed from C28; symbol Device:C_Small -> Roverette-rescue:C_Small-Device
- Q1, Q2: symbol Transistor_FET:BSS138 -> Roverette-rescue:BSS138-Transistor_FET
- U9: renamed from U11; symbol Interface_USB:CH340G -> Roverette-rescue:CH340G-Interface_USB
- Y1: symbol Device:Crystal_GND24 -> Roverette-rescue:Crystal_GND24-Device
Changed lines of the file:
@@
 $Descr A4 11693 8268
 encoding utf-8
-Sheet 11 12
+Sheet 10 11
 Title "USB Comms"
 Date "2019-01-26"
@@
 $EndDescr
 $Comp
-L Interface_USB:CH340G U11
+L Roverette-rescue:CH340G-Interface_USB U9
 U 1 1 5C49ED4D
 P 5400 3850
-F 0 "U11" H 5439 4559 50  0000 L CNN
+F 0 "U9" H 5439 4559 50  0000 L CNN
 F 1 "CH340G" H 5439 4480 50  0000 L CNN
 F 2 "Package_SO:SOIC-16_3.9x9.9mm_P1.27mm" H 5450 3300 50  0001 L CNN
@@
 	5400 3100 5400 3200
 $Comp
-L power:GND #PWR077
+L Roverette-rescue:GND-power #PWR072
 U 1 1 5C4AE9B0
 P 5400 4450
-F 0 "#PWR077" H 5400 4200 50  0001 C CNN
+F 0 "#PWR072" H 5400 4200 50  0001 C CNN
 F 1 "GND" H 5405 4277 50  0000 C CNN
 F 2 "" H 5400 4450 50  0001 C CNN
@@
 $EndComp
 $Comp
-L Device:C_Small C27
+L Roverette-rescue:C_Small-Device C28
 U 1 1 5C4E63C1
 P 4500 3200
-F 0 "C27" H 4592 3246 50  0000 L CNN
+F 0 "C28" H 4592 3246 50  0000 L CNN
 F 1 "100nF" H 4592 3155 50  0000 L CNN
 F 2 "Capacitor_SMD:C_0805_2012Metric" H 4500 3200 50  0001 C CNN
@@
 $EndComp
 $Comp
-L power:GND #PWR075
+L Roverette-rescue:GND-power #PWR066
 U 1 1 5C4F66CE
 P 4500 3300
-F 0 "#PWR075" H 4500 3050 50  0001 C CNN
+F 0 "#PWR066" H 4500 3050 50  0001 C CNN
 F 1 "GND" H 4505 3127 50  0000 C CNN
 F 2 "" H 4500 3300 50  0001 C CNN
@@
 $EndComp
 $Comp
-L Device:C_Small C28
+L Roverette-rescue:C_Small-Device C30
 U 1 1 5C4F6836
 P 5150 3200
-F 0 "C28" V 4921 3200 50  0000 C CNN
+F 0 "C30" V 4921 3200 50  0000 C CNN
 F 1 "10nF" V 5012 3200 50  0000 C CNN
 F 2 "Capacitor_SMD:C_0805_2012Metric" H 5150 3200 50  0001 C CNN
@@
 $EndComp
 $Comp
-L power:GND #PWR073
+L Roverette-rescue:GND-power #PWR070
 U 1 1 5C4F68F9
 P 5000 3250
-F 0 "#PWR073" H 5000 3000 50  0001 C CNN
+F 0 "#PWR070" H 5000 3000 50  0001 C CNN
 F 1 "GND" H 5005 3077 50  0000 C CNN
 F 2 "" H 5000 3250 50  0001 C CNN
@@
 NoConn ~ 5800 3750
 $Comp
-L power:+3.3V #PWR072
+L Roverette-rescue:+3.3V-power #PWR071
 U 1 1 5C8F955A
 P 5400 3100
-F 0 "#PWR072" H 5400 2950 50  0001 C CNN
+F 0 "#PWR071" H 5400 2950 50  0001 C CNN
 F 1 "+3.3V" H 5415 3273 50  0000 C CNN
 F 2 "" H 5400 3100 50  0001 C CNN
@@
 $EndComp
 $Comp
-L power:+3.3V #PWR071
+L Roverette-rescue:+3.3V-power #PWR065
 U 1 1 5C8F9686
 P 4500 3100
-F 0 "#PWR071" H 4500 2950 50  0001 C CNN
+F 0 "#PWR065" H 4500 2950 50  0001 C CNN
 F 1 "+3.3V" H 4515 3273 50  0000 C CNN
 F 2 "" H 4500 3100 50  0001 C CNN
@@
 Connection ~ 5300 3200
 $Comp
-L Transistor_FET:BSS138 Q1
+L Roverette-rescue:BSS138-Transistor_FET Q1
 U 1 1 5C9137B2
 P 6650 3850
@@
 $EndComp
 $Comp
-L Transistor_FET:BSS138 Q2
+L Roverette-rescue:BSS138-Transistor_FET Q2
 U 1 1 5C98AA01
 P 6650 4300
@@
 EN
 $Comp
-L power:GND #PWR076
+L Roverette-rescue:GND-power #PWR067
 U 1 1 5C908D2A
 P 4550 4250
-F 0 "#PWR076" H 4550 4000 50  0001 C CNN
+F 0 "#PWR067" H 4550 4000 50  0001 C CNN
 F 1 "GND" H 4555 4077 50  0001 C CNN
 F 2 "" H 4550 4250 50  0001 C CNN
@@
 $EndComp
 $Comp
-L Device:Crystal_GND24 Y1
+L Roverette-rescue:Crystal_GND24-Device Y1
 U 1 1 5C575BDD
 P 4550 4450
@@
 $EndComp
 $Comp
-L power:GND #PWR080
+L Roverette-rescue:GND-power #PWR069
 U 1 1 5C67ADA4
 P 4750 4700
-F 0 "#PWR080" H 4750 4450 50  0001 C CNN
+F 0 "#PWR069" H 4750 4450 50  0001 C CNN
 F 1 "GND" H 4755 4527 50  0000 C CNN
 F 2 "" H 4750 4700 50  0001 C CNN
@@
 $EndComp
 $Comp
-L power:GND #PWR079
+L Roverette-rescue:GND-power #PWR064
 U 1 1 5C67AD2C
 P 4350 4700
-F 0 "#PWR079" H 4350 4450 50  0001 C CNN
+F 0 "#PWR064" H 4350 4450 50  0001 C CNN
 F 1 "GND" H 4355 4527 50  0000 C CNN
 F 2 "" H 4350 4700 50  0001 C CNN
@@
 $EndComp
 $Comp
-L Device:C_Small C30
+L Roverette-rescue:C_Small-Device C29
 U 1 1 5C5B35D8
 P 4750 4600
-F 0 "C30" H 4842 4646 50  0000 L CNN
+F 0 "C29" H 4842 4646 50  0000 L CNN
 F 1 "22pF" H 4842 4555 50  0000 L CNN
 F 2 "Capacitor_SMD:C_0805_2012Metric" H 4750 4600 50  0001 C CNN
@@
 $EndComp
 $Comp
-L Device:C_Small C29
+L Roverette-rescue:C_Small-Device C27
 U 1 1 5C5B3556
 P 4350 4600
-F 0 "C29" H 4100 4600 50  0000 L CNN
+F 0 "C27" H 4100 4600 50  0000 L CNN
 F 1 "22pF" H 4100 4500 50  0000 L CNN
 F 2 "Capacitor_SMD:C_0805_2012Metric" H 4350 4600 50  0001 C CNN
@@
 $EndComp
 $Comp
-L power:+3.3V #PWR070
+L Roverette-rescue:+3.3V-power #PWR062
 U 1 1 5C8F971C
 P 4050 3100
-F 0 "#PWR070" H 4050 2950 50  0001 C CNN
+F 0 "#PWR062" H 4050 2950 50  0001 C CNN
 F 1 "+3.3V" H 4065 3273 50  0000 C CNN
 F 2 "" H 4050 3100 50  0001 C CNN
@@
 $EndComp
 $Comp
-L power:GND #PWR074
+L Roverette-rescue:GND-power #PWR063
 U 1 1 5C4F665E
 P 4050 3300
-F 0 "#PWR074" H 4050 3050 50  0001 C CNN
+F 0 "#PWR063" H 4050 3050 50  0001 C CNN
 F 1 "GND" H 4055 3127 50  0000 C CNN
 F 2 "" H 4050 3300 50  0001 C CNN
@@
 $EndComp
 $Comp
-L Device:CP_Small C?
+L Roverette-rescue:CP_Small-Device C?
 U 1 1 5DF9E1BC
 P 4050 3200
@@
 O2
 $Comp
-L power:GND #PWR078
+L Roverette-rescue:GND-power #PWR068
 U 1 1 608078C5
 P 4550 4650
-F 0 "#PWR078" H 4550 4400 50  0001 C CNN
+F 0 "#PWR068" H 4550 4400 50  0001 C CNN
 F 1 "GND" H 4555 4477 50  0001 C CNN
 F 2 "" H 4550 4650 50  0001 C CNN
