File: Hardware/Regulator.sch (KiCad schematic (older format))
At the start: 10 parts, among them U8 TPS56628

Commit message: Schematic updated, USB comms circuit added
Parts:
- D4: footprint (none) -> LED_SMD:LED_0805_2012Metric
- renumbered R26 to R29, U8 to U9
Changed lines of the file:
@@
 $Descr A4 11693 8268
 encoding utf-8
-Sheet 9 9
+Sheet 10 11
 Title ""
 Date ""
@@
 AR Path="/5FF19FBA" Ref="C?"  Part="1"
 AR Path="/5FF0069C/5FF19FBA" Ref="C18"  Part="1"
-F 0 "C18" H 4638 3696 50  0000 L CNN
+AR Path="/6071DAA9/5FF19FBA" Ref="C23"  Part="1"
+F 0 "C23" H 4638 3696 50  0000 L CNN
 F 1 "220nF" H 4638 3605 50  0000 L CNN
 F 2 "Capacitor_Tantalum_SMD:CP_EIA-3216-18_Kemet-A" H 4550 3650 50  0001 C CNN
@@
 AR Path="/5FF19FC0" Ref="C?"  Part="1"
 AR Path="/5FF0069C/5FF19FC0" Ref="C17"  Part="1"
-F 0 "C17" H 4238 3696 50  0000 L CNN
+AR Path="/6071DAA9/5FF19FC0" Ref="C22"  Part="1"
+F 0 "C22" H 4238 3696 50  0000 L CNN
 F 1 "4.7uF" H 4238 3605 50  0000 L CNN
 F 2 "Capacitor_Tantalum_SMD:CP_EIA-3528-15_AVX-H" H 4150 3650 50  0001 C CNN
@@
 AR Path="/5FF19FC7" Ref="L?"  Part="1"
 AR Path="/5FF0069C/5FF19FC7" Ref="L2"  Part="1"
-F 0 "L2" V 6835 3400 50  0000 C CNN
+AR Path="/6071DAA9/5FF19FC7" Ref="L3"  Part="1"
+F 0 "L3" V 6835 3400 50  0000 C CNN
 F 1 "15uH" V 6744 3400 50  0000 C CNN
 F 2 "Inductor_SMD:L_Neosid_SMs42" H 6650 3400 50  0001 C CNN
@@
 AR Path="/5FF19FCD" Ref="C?"  Part="1"
 AR Path="/5FF0069C/5FF19FCD" Ref="C16"  Part="1"
-F 0 "C16" V 5971 3400 50  0000 C CNN
+AR Path="/6071DAA9/5FF19FCD" Ref="C21"  Part="1"
+F 0 "C21" V 5971 3400 50  0000 C CNN
 F 1 "100nF" V 6062 3400 50  0000 C CNN
 F 2 "Capacitor_SMD:C_0805_2012Metric" H 6200 3400 50  0001 C CNN
@@
 P 4150 3350
 AR Path="/5FF19FDD" Ref="#PWR?"  Part="1"
-AR Path="/5FF0069C/5FF19FDD" Ref="#PWR057"  Part="1"
-F 0 "#PWR057" H 4150 3200 50  0001 C CNN
+AR Path="/5FF0069C/5FF19FDD" Ref="#PWR066"  Part="1"
+AR Path="/6071DAA9/5FF19FDD" Ref="#PWR068"  Part="1"
+F 0 "#PWR068" H 4150 3200 50  0001 C CNN
 F 1 "+BATT" H 4165 3523 50  0000 C CNN
 F 2 "" H 4150 3350 50  0001 C CNN
@@
 P 5600 3950
 AR Path="/5FF1A004" Ref="#PWR?"  Part="1"
-AR Path="/5FF0069C/5FF1A004" Ref="#PWR058"  Part="1"
-F 0 "#PWR058" H 5600 3700 50  0001 C CNN
+AR Path="/5FF0069C/5FF1A004" Ref="#PWR067"  Part="1"
+AR Path="/6071DAA9/5FF1A004" Ref="#PWR069"  Part="1"
+F 0 "#PWR069" H 5600 3700 50  0001 C CNN
 F 1 "GND" H 5605 3777 50  0000 C CNN
 F 2 "" H 5600 3950 50  0001 C CNN
@@
 P 5600 3300
 AR Path="/5FF1A031" Ref="U?"  Part="1"
-AR Path="/5FF0069C/5FF1A031" Ref="U8"  Part="1"
-F 0 "U8" H 5600 3465 50  0000 C CNN
+AR Path="/5FF0069C/5FF1A031" Ref="U9"  Part="1"
+AR Path="/6071DAA9/5FF1A031" Ref="U10"  Part="1"
+F 0 "U10" H 5600 3465 50  0000 C CNN
 F 1 "TPS56628" H 5600 3374 50  0000 C CNN
 F 2 "Package_SO:HSOP-8-1EP_3.9x4.9mm_P1.27mm_EP2.41x3.1mm_ThermalVias" H 5600 3450 50  0001 C CNN
@@
 AR Path="/5FF1A03A" Ref="D?"  Part="1"
 AR Path="/5FF0069C/5FF1A03A" Ref="D4"  Part="1"
-F 0 "D4" H 4950 3800 50  0000 C CNN
+AR Path="/6071DAA9/5FF1A03A" Ref="D6"  Part="1"
+F 0 "D6" H 4950 3800 50  0000 C CNN
 F 1 "GREEN" H 5150 3800 50  0000 C CNN
-F 2 "" V 5050 3700 50  0001 C CNN
+F 2 "LED_SMD:LED_0805_2012Metric" V 5050 3700 50  0001 C CNN
 F 3 "~" V 5050 3700 50  0001 C CNN
 	1    5050 3700
@@
 AR Path="/5EA2026E/5FF1A040" Ref="R?"  Part="1"
 AR Path="/5FF1A040" Ref="R?"  Part="1"
-AR Path="/5FF0069C/5FF1A040" Ref="R26"  Part="1"
-F 0 "R26" V 5150 3650 50  0000 L CNN
+AR Path="/5FF0069C/5FF1A040" Ref="R29"  Part="1"
+AR Path="/6071DAA9/5FF1A040" Ref="R30"  Part="1"
+F 0 "R30" V 5150 3650 50  0000 L CNN
 F 1 "4.7k" V 5100 3500 50  0000 L CNN
 F 2 "Resistor_SMD:R_0805_2012Metric" H 5050 3600 50  0001 C CNN
@@
 AR Path="/5FF1A05B" Ref="C?"  Part="1"
 AR Path="/5FF0069C/5FF1A05B" Ref="C19"  Part="1"
-F 0 "C19" H 6938 3696 50  0000 L CNN
+AR Path="/6071DAA9/5FF1A05B" Ref="C24"  Part="1"
+F 0 "C24" H 6938 3696 50  0000 L CNN
 F 1 "100uF" H 6938 3605 50  0000 L CNN
 F 2 "Capacitor_Tantalum_SMD:CP_EIA-7343-31_Kemet-D" H 6850 3650 50  0001 C CNN
@@
 AR Path="/5FF1A061" Ref="C?"  Part="1"
 AR Path="/5FF0069C/5FF1A061" Ref="C20"  Part="1"
-F 0 "C20" H 7338 3696 50  0000 L CNN
+AR Path="/6071DAA9/5FF1A061" Ref="C25"  Part="1"
+F 0 "C25" H 7338 3696 50  0000 L CNN
 F 1 "4.7uF" H 7338 3605 50  0000 L CNN
 F 2 "Capacitor_Tantalum_SMD:CP_EIA-3528-15_AVX-H" H 7250 3650 50  0001 C CNN
@@
 AR Path="/5FF1A067" Ref="D?"  Part="1"
 AR Path="/5FF0069C/5FF1A067" Ref="D3"  Part="1"
-F 0 "D3" V 6404 3729 50  0000 L CNN
+AR Path="/6071DAA9/5FF1A067" Ref="D5"  Part="1"
+F 0 "D5" V 6404 3729 50  0000 L CNN
 F 1 "5A" V 6495 3729 50  0000 L CNN
 F 2 "Diode_SMD:D_SOD-123F" V 6450 3650 50  0001 C CNN
@@
 Wire Wire Line
 	4150 3400 4100 3400
-Wire Wire Line
-	7250 3350 7250 3400
-$Comp
-L power:PWR_FLAG #FLG?
-U 1 1 6071CB78
+Text HLabel 6050 3700 2    50   Input ~ 0
+SNS
+Wire Wire Line
+	7300 3400 7250 3400
+$Comp
+L power:PWR_FLAG #FLG0102
+U 1 1 608831A8
 P 7250 3350
-AR Path="/6071CB78" Ref="#FLG?"  Part="1"
-AR Path="/5FF0069C/6071CB78" Ref="#FLG0103"  Part="1"
-F 0 "#FLG0103" H 7250 3425 50  0001 C CNN
+AR Path="/6071DAA9/608831A8" Ref="#FLG0102"  Part="1"
+AR Path="/5FF0069C/608831A8" Ref="#FLG0101"  Part="1"
+F 0 "#FLG0102" H 7250 3425 50  0001 C CNN
 F 1 "PWR_FLAG" H 7250 3523 50  0000 C CNN
 F 2 "" H 7250 3350 50  0001 C CNN
@@
 	1    0    0    -1
 $EndComp
-Text HLabel 6050 3700 2    50   Input ~ 0
-SNS
-Wire Wire Line
-	7300 3400 7250 3400
+Wire Wire Line
+	7250 3350 7250 3400
 $EndSCHEMATC

Commit message: PCB design started
Parts:
- C16: renamed from C17; symbol Device:CP_Small -> Roverette-rescue:CP_Small-Device
- C17: renamed from C18; symbol Device:CP_Small -> Roverette-rescue:CP_Small-Device
- C18: renamed from C16; symbol Device:C_Small -> Roverette-rescue:C_Small-Device
- C19, C20: symbol Device:CP_Small -> Roverette-rescue:CP_Small-Device
- D3: renamed from D4; symbol Device:LED_Small -> Roverette-rescue:LED_Small-Device
- D4: renamed from D3; symbol Device:D_Schottky -> Roverette-rescue:D_Schottky-Device
- L2: symbol Device:L_Small -> Roverette-rescue:L_Small-Device
- R29: symbol Device:R_Small_US -> Roverette-rescue:R_Small_US-Device
- renumbered U9 to U7
Changed lines of the file:
@@
 $Descr A4 11693 8268
 encoding utf-8
-Sheet 10 12
+Sheet 8 11
 Title ""
 Date ""
@@
 $EndDescr
 $Comp
-L Device:CP_Small C?
+L Roverette-rescue:CP_Small-Device C?
 U 1 1 5FF19FBA
 P 4550 3650
 AR Path="/5E9DAA7B/5FF19FBA" Ref="C?"  Part="1"
 AR Path="/5FF19FBA" Ref="C?"  Part="1"
-AR Path="/5FF0069C/5FF19FBA" Ref="C18"  Part="1"
-AR Path="/6071DAA9/5FF19FBA" Ref="C23"  Part="1"
-F 0 "C23" H 4638 3696 50  0000 L CNN
+AR Path="/5FF0069C/5FF19FBA" Ref="C17"  Part="1"
+AR Path="/6071DAA9/5FF19FBA" Ref="C22"  Part="1"
+F 0 "C17" H 4638 3696 50  0000 L CNN
 F 1 "220nF" H 4638 3605 50  0000 L CNN
 F 2 "Capacitor_Tantalum_SMD:CP_EIA-3216-18_Kemet-A" H 4550 3650 50  0001 C CNN
@@
 $EndComp
 $Comp
-L Device:CP_Small C?
+L Roverette-rescue:CP_Small-Device C?
 U 1 1 5FF19FC0
 P 4150 3650
 AR Path="/5E9DAA7B/5FF19FC0" Ref="C?"  Part="1"
 AR Path="/5FF19FC0" Ref="C?"  Part="1"
-AR Path="/5FF0069C/5FF19FC0" Ref="C17"  Part="1"
-AR Path="/6071DAA9/5FF19FC0" Ref="C22"  Part="1"
-F 0 "C22" H 4238 3696 50  0000 L CNN
+AR Path="/5FF0069C/5FF19FC0" Ref="C16"  Part="1"
+AR Path="/6071DAA9/5FF19FC0" Ref="C21"  Part="1"
+F 0 "C16" H 4238 3696 50  0000 L CNN
 F 1 "4.7uF" H 4238 3605 50  0000 L CNN
 F 2 "Capacitor_Tantalum_SMD:CP_EIA-3528-15_AVX-H" H 4150 3650 50  0001 C CNN
@@
 $EndComp
 $Comp
-L Device:L_Small L?
+L Roverette-rescue:L_Small-Device L?
 U 1 1 5FF19FC7
 P 6650 3400
@@
 AR Path="/5FF0069C/5FF19FC7" Ref="L2"  Part="1"
 AR Path="/6071DAA9/5FF19FC7" Ref="L3"  Part="1"
-F 0 "L3" V 6835 3400 50  0000 C CNN
+F 0 "L2" V 6835 3400 50  0000 C CNN
 F 1 "15uH" V 6744 3400 50  0000 C CNN
 F 2 "Inductor_SMD:L_Neosid_SMs42" H 6650 3400 50  0001 C CNN
@@
 $EndComp
 $Comp
-L Device:C_Small C?
+L Roverette-rescue:C_Small-Device C?
 U 1 1 5FF19FCD
 P 6200 3400
 AR Path="/5E9DAA7B/5FF19FCD" Ref="C?"  Part="1"
 AR Path="/5FF19FCD" Ref="C?"  Part="1"
-AR Path="/5FF0069C/5FF19FCD" Ref="C16"  Part="1"
-AR Path="/6071DAA9/5FF19FCD" Ref="C21"  Part="1"
-F 0 "C21" V 5971 3400 50  0000 C CNN
+AR Path="/5FF0069C/5FF19FCD" Ref="C18"  Part="1"
+AR Path="/6071DAA9/5FF19FCD" Ref="C23"  Part="1"
+F 0 "C18" V 5971 3400 50  0000 C CNN
 F 1 "100nF" V 6062 3400 50  0000 C CNN
 F 2 "Capacitor_SMD:C_0805_2012Metric" H 6200 3400 50  0001 C CNN
@@
 	6450 3400 6550 3400
 $Comp
-L power:+BATT #PWR?
+L Roverette-rescue:+BATT-power #PWR?
 U 1 1 5FF19FDD
 P 4150 3350
 AR Path="/5FF19FDD" Ref="#PWR?"  Part="1"
-AR Path="/5FF0069C/5FF19FDD" Ref="#PWR066"  Part="1"
-AR Path="/6071DAA9/5FF19FDD" Ref="#PWR068"  Part="1"
-F 0 "#PWR068" H 4150 3200 50  0001 C CNN
+AR Path="/5FF0069C/5FF19FDD" Ref="#PWR058"  Part="1"
+AR Path="/6071DAA9/5FF19FDD" Ref="#PWR060"  Part="1"
+F 0 "#PWR058" H 4150 3200 50  0001 C CNN
 F 1 "+BATT" H 4165 3523 50  0000 C CNN
 F 2 "" H 4150 3350 50  0001 C CNN
@@
 Connection ~ 7250 3400
 $Comp
-L power:GND #PWR?
+L Roverette-rescue:GND-power #PWR?
 U 1 1 5FF1A004
 P 5600 3950
 AR Path="/5FF1A004" Ref="#PWR?"  Part="1"
-AR Path="/5FF0069C/5FF1A004" Ref="#PWR067"  Part="1"
-AR Path="/6071DAA9/5FF1A004" Ref="#PWR069"  Part="1"
-F 0 "#PWR069" H 5600 3700 50  0001 C CNN
+AR Path="/5FF0069C/5FF1A004" Ref="#PWR059"  Part="1"
+AR Path="/6071DAA9/5FF1A004" Ref="#PWR061"  Part="1"
+F 0 "#PWR059" H 5600 3700 50  0001 C CNN
 F 1 "GND" H 5605 3777 50  0000 C CNN
 F 2 "" H 5600 3950 50  0001 C CNN
@@
 P 5600 3300
 AR Path="/5FF1A031" Ref="U?"  Part="1"
-AR Path="/5FF0069C/5FF1A031" Ref="U9"  Part="1"
-AR Path="/6071DAA9/5FF1A031" Ref="U10"  Part="1"
-F 0 "U10" H 5600 3465 50  0000 C CNN
+AR Path="/5FF0069C/5FF1A031" Ref="U7"  Part="1"
+AR Path="/6071DAA9/5FF1A031" Ref="U8"  Part="1"
+F 0 "U7" H 5600 3465 50  0000 C CNN
 F 1 "TPS56628" H 5600 3374 50  0000 C CNN
 F 2 "Package_SO:HSOP-8-1EP_3.9x4.9mm_P1.27mm_EP2.41x3.1mm_ThermalVias" H 5600 3450 50  0001 C CNN
@@
 	5100 3400 5150 3400
 $Comp
-L Device:LED_Small D?
+L Roverette-rescue:LED_Small-Device D?
 U 1 1 5FF1A03A
 P 5050 3700
 AR Path="/5FF1A03A" Ref="D?"  Part="1"
-AR Path="/5FF0069C/5FF1A03A" Ref="D4"  Part="1"
-AR Path="/6071DAA9/5FF1A03A" Ref="D6"  Part="1"
-F 0 "D6" H 4950 3800 50  0000 C CNN
+AR Path="/5FF0069C/5FF1A03A" Ref="D3"  Part="1"
+AR Path="/6071DAA9/5FF1A03A" Ref="D5"  Part="1"
+F 0 "D3" H 4950 3800 50  0000 C CNN
 F 1 "GREEN" H 5150 3800 50  0000 C CNN
 F 2 "LED_SMD:LED_0805_2012Metric" V 5050 3700 50  0001 C CNN
@@
 $EndComp
 $Comp
-L Device:R_Small_US R?
+L Roverette-rescue:R_Small_US-Device R?
 U 1 1 5FF1A040
 P 5050 3600
@@
 AR Path="/5FF0069C/5FF1A040" Ref="R29"  Part="1"
 AR Path="/6071DAA9/5FF1A040" Ref="R30"  Part="1"
-F 0 "R30" V 5150 3650 50  0000 L CNN
+F 0 "R29" V 5150 3650 50  0000 L CNN
 F 1 "4.7k" V 5100 3500 50  0000 L CNN
 F 2 "Resistor_SMD:R_0805_2012Metric" H 5050 3600 50  0001 C CNN
@@
 	4550 3750 4550 3900
 $Comp
-L Device:CP_Small C?
+L Roverette-rescue:CP_Small-Device C?
 U 1 1 5FF1A05B
 P 6850 3650
@@
 AR Path="/5FF0069C/5FF1A05B" Ref="C19"  Part="1"
 AR Path="/6071DAA9/5FF1A05B" Ref="C24"  Part="1"
-F 0 "C24" H 6938 3696 50  0000 L CNN
+F 0 "C19" H 6938 3696 50  0000 L CNN
 F 1 "100uF" H 6938 3605 50  0000 L CNN
 F 2 "Capacitor_Tantalum_SMD:CP_EIA-7343-31_Kemet-D" H 6850 3650 50  0001 C CNN
@@
 $EndComp
 $Comp
-L Device:CP_Small C?
+L Roverette-rescue:CP_Small-Device C?
 U 1 1 5FF1A061
 P 7250 3650
@@
 AR Path="/5FF0069C/5FF1A061" Ref="C20"  Part="1"
 AR Path="/6071DAA9/5FF1A061" Ref="C25"  Part="1"
-F 0 "C25" H 7338 3696 50  0000 L CNN
+F 0 "C20" H 7338 3696 50  0000 L CNN
 F 1 "4.7uF" H 7338 3605 50  0000 L CNN
 F 2 "Capacitor_Tantalum_SMD:CP_EIA-3528-15_AVX-H" H 7250 3650 50  0001 C CNN
@@
 $EndComp
 $Comp
-L Device:D_Schottky D?
+L Roverette-rescue:D_Schottky-Device D?
 U 1 1 5FF1A067
 P 6450 3650
 AR Path="/5E9DAA7B/5FF1A067" Ref="D?"  Part="1"
 AR Path="/5FF1A067" Ref="D?"  Part="1"
-AR Path="/5FF0069C/5FF1A067" Ref="D3"  Part="1"
-AR Path="/6071DAA9/5FF1A067" Ref="D5"  Part="1"
-F 0 "D5" V 6404 3729 50  0000 L CNN
+AR Path="/5FF0069C/5FF1A067" Ref="D4"  Part="1"
+AR Path="/6071DAA9/5FF1A067" Ref="D6"  Part="1"
+F 0 "D4" V 6404 3729 50  0000 L CNN
 F 1 "5A" V 6495 3729 50  0000 L CNN
 F 2 "Diode_SMD:D_SOD-123F" V 6450 3650 50  0001 C CNN
@@
 Wire Wire Line
 	7300 3400 7250 3400
-$Comp
-L power:PWR_FLAG #FLG0102
-U 1 1 608831A8
-P 7250 3350
-AR Path="/6071DAA9/608831A8" Ref="#FLG0102"  Part="1"
-AR Path="/5FF0069C/608831A8" Ref="#FLG0101"  Part="1"
-F 0 "#FLG0102" H 7250 3425 50  0001 C CNN
-F 1 "PWR_FLAG" H 7250 3523 50  0000 C CNN
-F 2 "" H 7250 3350 50  0001 C CNN
-F 3 "~" H 7250 3350 50  0001 C CNN
-	1    7250 3350
-	1    0    0    -1
-$EndComp
-Wire Wire Line
-	7250 3350 7250 3400
 $EndSCHEMATC

Commit message: Did placements and routing of one regulator
Connections:
- net sw: now reaches C18.1, D4.1 (K), L2.1, U7.6 (SW)
Other:
- moved on the sheet: C21, C22
Changed lines of the file:
@@
 $Descr A4 11693 8268
 encoding utf-8
-Sheet 8 11
+Sheet 9 11
 Title ""
 Date ""
@@
 L Roverette-rescue:CP_Small-Device C?
 U 1 1 5FF19FBA
-P 4550 3650
+P 4450 3650
 AR Path="/5E9DAA7B/5FF19FBA" Ref="C?"  Part="1"
 AR Path="/5FF19FBA" Ref="C?"  Part="1"
 AR Path="/5FF0069C/5FF19FBA" Ref="C17"  Part="1"
 AR Path="/6071DAA9/5FF19FBA" Ref="C22"  Part="1"
-F 0 "C17" H 4638 3696 50  0000 L CNN
-F 1 "220nF" H 4638 3605 50  0000 L CNN
-F 2 "Capacitor_Tantalum_SMD:CP_EIA-3216-18_Kemet-A" H 4550 3650 50  0001 C CNN
-F 3 "~" H 4550 3650 50  0001 C CNN
-	1    4550 3650
+F 0 "C22" H 4538 3696 50  0000 L CNN
+F 1 "220nF" H 4538 3605 50  0000 L CNN
+F 2 "Capacitor_Tantalum_SMD:CP_EIA-3216-18_Kemet-A" H 4450 3650 50  0001 C CNN
+F 3 "~" H 4450 3650 50  0001 C CNN
+	1    4450 3650
 	1    0    0    -1
 $EndComp
@@
 L Roverette-rescue:CP_Small-Device C?
 U 1 1 5FF19FC0
-P 4150 3650
+P 4050 3650
 AR Path="/5E9DAA7B/5FF19FC0" Ref="C?"  Part="1"
 AR Path="/5FF19FC0" Ref="C?"  Part="1"
 AR Path="/5FF0069C/5FF19FC0" Ref="C16"  Part="1"
 AR Path="/6071DAA9/5FF19FC0" Ref="C21"  Part="1"
-F 0 "C16" H 4238 3696 50  0000 L CNN
-F 1 "4.7uF" H 4238 3605 50  0000 L CNN
-F 2 "Capacitor_Tantalum_SMD:CP_EIA-3528-15_AVX-H" H 4150 3650 50  0001 C CNN
-F 3 "~" H 4150 3650 50  0001 C CNN
-	1    4150 3650
+F 0 "C21" H 4138 3696 50  0000 L CNN
+F 1 "4.7uF" H 4138 3605 50  0000 L CNN
+F 2 "Capacitor_Tantalum_SMD:CP_EIA-3528-15_AVX-H" H 4050 3650 50  0001 C CNN
+F 3 "~" H 4050 3650 50  0001 C CNN
+	1    4050 3650
 	1    0    0    -1
 $EndComp
@@
 AR Path="/5FF0069C/5FF19FC7" Ref="L2"  Part="1"
 AR Path="/6071DAA9/5FF19FC7" Ref="L3"  Part="1"
-F 0 "L2" V 6835 3400 50  0000 C CNN
+F 0 "L3" V 6835 3400 50  0000 C CNN
 F 1 "15uH" V 6744 3400 50  0000 C CNN
 F 2 "Inductor_SMD:L_Neosid_SMs42" H 6650 3400 50  0001 C CNN
@@
 AR Path="/5FF0069C/5FF19FCD" Ref="C18"  Part="1"
 AR Path="/6071DAA9/5FF19FCD" Ref="C23"  Part="1"
-F 0 "C18" V 5971 3400 50  0000 C CNN
+F 0 "C23" V 5971 3400 50  0000 C CNN
 F 1 "100nF" V 6062 3400 50  0000 C CNN
 F 2 "Capacitor_SMD:C_0805_2012Metric" H 6200 3400 50  0001 C CNN
@@
 Connection ~ 6450 3400
 Wire Wire Line
-	4150 3400 4550 3400
-Connection ~ 4550 3400
+	4050 3400 4450 3400
+Connection ~ 4450 3400
 Wire Wire Line
 	6450 3400 6550 3400
@@
 L Roverette-rescue:+BATT-power #PWR?
 U 1 1 5FF19FDD
-P 4150 3350
+P 4050 3350
 AR Path="/5FF19FDD" Ref="#PWR?"  Part="1"
 AR Path="/5FF0069C/5FF19FDD" Ref="#PWR058"  Part="1"
 AR Path="/6071DAA9/5FF19FDD" Ref="#PWR060"  Part="1"
-F 0 "#PWR058" H 4150 3200 50  0001 C CNN
-F 1 "+BATT" H 4165 3523 50  0000 C CNN
-F 2 "" H 4150 3350 50  0001 C CNN
-F 3 "" H 4150 3350 50  0001 C CNN
-	1    4150 3350
-	1    0    0    -1
-$EndComp
-Wire Wire Line
-	4150 3350 4150 3400
-Connection ~ 4150 3400
+F 0 "#PWR060" H 4050 3200 50  0001 C CNN
+F 1 "+BATT" H 4065 3523 50  0000 C CNN
+F 2 "" H 4050 3350 50  0001 C CNN
+F 3 "" H 4050 3350 50  0001 C CNN
+	1    4050 3350
+	1    0    0    -1
+$EndComp
+Wire Wire Line
+	4050 3350 4050 3400
+Connection ~ 4050 3400
 Wire Wire Line
 	6850 3400 7250 3400
@@
 AR Path="/5FF0069C/5FF1A004" Ref="#PWR059"  Part="1"
 AR Path="/6071DAA9/5FF1A004" Ref="#PWR061"  Part="1"
-F 0 "#PWR059" H 5600 3700 50  0001 C CNN
+F 0 "#PWR061" H 5600 3700 50  0001 C CNN
 F 1 "GND" H 5605 3777 50  0000 C CNN
 F 2 "" H 5600 3950 50  0001 C CNN
@@
 Text Notes 7350 3800 0    50   ~ 0
 Tant
-Text Notes 4250 3800 0    50   ~ 0
-Tant
-Text Notes 4650 3800 0    50   ~ 0
+Text Notes 4150 3800 0    50   ~ 0
+Tant
+Text Notes 4550 3800 0    50   ~ 0
 Tant
 $Comp
@@
 AR Path="/5FF0069C/5FF1A031" Ref="U7"  Part="1"
 AR Path="/6071DAA9/5FF1A031" Ref="U8"  Part="1"
-F 0 "U7" H 5600 3465 50  0000 C CNN
+F 0 "U8" H 5600 3465 50  0000 C CNN
 F 1 "TPS56628" H 5600 3374 50  0000 C CNN
 F 2 "Package_SO:HSOP-8-1EP_3.9x4.9mm_P1.27mm_EP2.41x3.1mm_ThermalVias" H 5600 3450 50  0001 C CNN
@@
 	1    0    0    -1
 $EndComp
-Wire Wire Line
-	5150 3500 5100 3500
-Wire Wire Line
-	5100 3500 5100 3400
-Wire Wire Line
-	5100 3400 5150 3400
 $Comp
 L Roverette-rescue:LED_Small-Device D?
@@
 AR Path="/5FF0069C/5FF1A03A" Ref="D3"  Part="1"
 AR Path="/6071DAA9/5FF1A03A" Ref="D5"  Part="1"
-F 0 "D3" H 4950 3800 50  0000 C CNN
+F 0 "D5" H 4950 3800 50  0000 C CNN
 F 1 "GREEN" H 5150 3800 50  0000 C CNN
 F 2 "LED_SMD:LED_0805_2012Metric" V 5050 3700 50  0001 C CNN
@@
 AR Path="/5FF0069C/5FF1A040" Ref="R29"  Part="1"
 AR Path="/6071DAA9/5FF1A040" Ref="R30"  Part="1"
-F 0 "R29" V 5150 3650 50  0000 L CNN
-F 1 "4.7k" V 5100 3500 50  0000 L CNN
+F 0 "R30" V 5200 3650 50  0000 L CNN
+F 1 "4.7k" V 5100 3650 50  0000 L CNN
 F 2 "Resistor_SMD:R_0805_2012Metric" H 5050 3600 50  0001 C CNN
 F 3 "https://lcsc.com/product-detail/Chip-Resistor-Surface-Mount_Uniroyal-Elec-0805W8F1002T5E_C17414.html/?href=jlc-SMT" H 5050 3600 50  0001 C CNN
@@
 	4900 3700 4950 3700
 Wire Wire Line
-	4550 3400 5100 3400
-Connection ~ 5100 3400
-Wire Wire Line
 	6350 3400 6350 3550
 Connection ~ 5600 3900
 Wire Wire Line
-	4550 3900 5600 3900
-Wire Wire Line
-	4550 3400 4550 3550
-Wire Wire Line
-	4150 3400 4150 3550
+	4450 3400 4450 3550
+Wire Wire Line
+	4050 3400 4050 3550
 Wire Wire Line
 	5600 3900 6450 3900
-Connection ~ 4550 3900
+Connection ~ 4450 3900
 Connection ~ 6450 3900
 Wire Wire Line
-	4150 3750 4150 3900
-Wire Wire Line
-	4150 3900 4550 3900
-Wire Wire Line
-	4550 3750 4550 3900
+	4050 3750 4050 3900
+Wire Wire Line
+	4050 3900 4450 3900
+Wire Wire Line
+	4450 3750 4450 3900
 $Comp
 L Roverette-rescue:CP_Small-Device C?
@@
 AR Path="/5FF0069C/5FF1A05B" Ref="C19"  Part="1"
 AR Path="/6071DAA9/5FF1A05B" Ref="C24"  Part="1"
-F 0 "C19" H 6938 3696 50  0000 L CNN
+F 0 "C24" H 6938 3696 50  0000 L CNN
 F 1 "100uF" H 6938 3605 50  0000 L CNN
 F 2 "Capacitor_Tantalum_SMD:CP_EIA-7343-31_Kemet-D" H 6850 3650 50  0001 C CNN
@@
 AR Path="/5FF0069C/5FF1A061" Ref="C20"  Part="1"
 AR Path="/6071DAA9/5FF1A061" Ref="C25"  Part="1"
-F 0 "C20" H 7338 3696 50  0000 L CNN
+F 0 "C25" H 7338 3696 50  0000 L CNN
 F 1 "4.7uF" H 7338 3605 50  0000 L CNN
 F 2 "Capacitor_Tantalum_SMD:CP_EIA-3528-15_AVX-H" H 7250 3650 50  0001 C CNN
@@
 AR Path="/5FF0069C/5FF1A067" Ref="D4"  Part="1"
 AR Path="/6071DAA9/5FF1A067" Ref="D6"  Part="1"
-F 0 "D4" V 6404 3729 50  0000 L CNN
+F 0 "D6" V 6404 3729 50  0000 L CNN
 F 1 "5A" V 6495 3729 50  0000 L CNN
 F 2 "Diode_SMD:D_SOD-123F" V 6450 3650 50  0001 C CNN
@@
 Wire Wire Line
 	6450 3800 6450 3900
-Text HLabel 4100 3400 0    50   Input ~ 0
+Text HLabel 4000 3400 0    50   Input ~ 0
 VBAT
 Text HLabel 7300 3400 2    50   Output ~ 0
 VOUT
 Wire Wire Line
-	4150 3400 4100 3400
+	4050 3400 4000 3400
 Text HLabel 6050 3700 2    50   Input ~ 0
 SNS
 Wire Wire Line
 	7300 3400 7250 3400
+Text Label 6100 3550 0    50   ~ 0
+sw
+Wire Wire Line
+	5100 3400 5150 3400
+Wire Wire Line
+	5100 3500 5100 3400
+Wire Wire Line
+	5150 3500 5100 3500
+Wire Wire Line
+	4450 3900 5600 3900
+Wire Wire Line
+	4450 3400 5100 3400
+Connection ~ 5100 3400
 $EndSCHEMATC
