File: Hardware/Roverette.kicad_pcb (KiCad board)
At the start: 2 copper layers, 94 parts, among them J1 USB_C_Receptacle, J2 HDR, M1 Motor_DC, M2 Motor_DC, Q1 BSS138, Q2 BSS138, SW1 SW_Push, SW2 SW_Push, U1 ESDA6V8AV5, U10 TPS56628, U11 CH340G, U2 DRV8874, U3 DRV8874, U4 CNY70, U5 CNY70, U6 ESP32-WROOM-32D, U7 MPU-9250, U8 BQ25616, U9 TPS56628, Y1 12MHz

Commit message: PCB design started
Parts:
- removed the J1 at (94.4, 103.5)
- removed the U1 at (113.3, 114.8)
- removed the U7 at (128.7, 117.8)
- added J2: USB_C_Receptacle, Connector_USB:USB_C_Receptacle_XKB_U262-16XN-4BVC11, F.Cu at (165.0, 95.0)
- added J3: JTAG, Connector_PinHeader_1.27mm:PinHeader_2x05_P1.27mm_Vertical_SMD, F.Cu at (98.0, 99.0)
- added U10: ESDA6V8AV5, Package_TO_SOT_SMD:SOT-553, F.Cu at (170.5, 86.5)
- J1: renamed from J2; footprint Connector_PinSocket_2.54mm:PinSocket_1x03_P2.54mm_Vertical -> Connector_PinHeader_2.54mm:PinHeader_1x03_P2.54mm_Vertical
- R21, R22: value 4.7k -> 50R
- moved C16 98.4 mm to (69.7, 94.7)
- moved C19 98.4 mm to (63.2, 88.9)
- moved C18 98.4 mm to (68.9, 98.4)
- moved D4 98.4 mm to (75.5, 97.4)
- moved U7 98.4 mm to (62.5, 95.1)
- moved C17 98.4 mm to (75.6, 94.1)
- moved C20 98.4 mm to (78.3, 88.2)
- moved D3 98.4 mm to (80.6, 91.9)
- moved L2 98.4 mm to (71.7, 89.3)
- moved R29 98.4 mm to (80.4, 97.2)
- moved BT1 76.2 mm to (149.0, 62.5)
- moved TP1 64.0 mm to (161.0, 57.0)
- moved D6 60.8 mm to (84.8, 126.1)
- moved U8 60.8 mm to (71.9, 123.8)
- moved C22 60.8 mm to (84.9, 122.9)
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- renumbered C3 to C1, C11 to C10, C9 to C11, C14 to C12, C12 to C13, C15 to C14, C13 to C15, C17 to C16, C18 to C17, C16 to C18, C4 to C2, C22 to C21, C23 to C22, C21 to C23, C29 to C27, C27 to C28, C30 to C29, C1 to C3, C28 to C30, C2 to C4, C7 to C5, C8 to C6, C5 to C7, C6 to C8, C10 to C9, D4 to D3, D3 to D4, D6 to D5, D5 to D6, R11 to R10, R10 to R11, R14 to R13, R15 to R14, R13 to R15, R17 to R16, R18 to R17, R16 to R18, R27 to R24, R24 to R25, R28 to R26, R25 to R27, R26 to R28, R7 to R6, R6 to R7, TP3 to TP1, TP1 to TP2, TP2 to TP3, U2 to U1, U3 to U2, U4 to U3, U5 to U4, U6 to U5, U8 to U6, U9 to U7, U10 to U8, U11 to U9
Connections:
- net Net-(U6-Pad17) renamed /MCU/SDH
- net Net-(U6-Pad18) renamed /MCU/SWP
- net Net-(U6-Pad19) renamed /MCU/SCS
- net Net-(U6-Pad20) renamed /MCU/SCK
- net Net-(U6-Pad21) renamed /MCU/SD0
- net Net-(U6-Pad22) renamed /MCU/SDI
- net Net-(U6-Pad7) renamed /MCU/IO35
- net Net-(U6-Pad8) renamed /MCU/IO32
- net Net-(U6-Pad9) renamed /MCU/IO33
- net VBUS renamed /Charger/VBUS
- R21 pad 2: /SCL -> Net-(R21-Pad2)
- R22 pad 2: /SDA -> Net-(R22-Pad2)
- U3 pad 3: +3V3 -> Net-(R21-Pad2)
- U4 pad 3: +3V3 -> Net-(R22-Pad2)
- U5 pad 10: /INT -> /PG
- U5 pad 11: /FSYNC -> /CHG
- U5 pad 12: Net-(U6-Pad12) (its old number) -> /MCU/IO27
- U5 pad 13: /FAULT_L -> /MCU/TCK
- U5 pad 14: /PH_L -> /MCU/TDO
- U5 pad 16: /SLEEP_L -> /MCU/TDI
- U5 pad 23: /FAULT_R -> /MCU/TMS
- U5 pad 31: /PG -> /PH_L
- U5 pad 33: /SDA -> /SLEEP_L
- U5 pad 36: /SCL -> /FAULT_L
- U5 pad 37: /CHG -> /FAULT_R
- U5 pad 6: Net-(U6-Pad6) (its old number) -> /MCU/IO34
- U9 pad 5: /D+ -> /USB C/D+
- U9 pad 6: /D- -> /USB C/D-

Commit message: Did placements and routing of one regulator
Parts:
- TP2: value TestPoint -> vDrive
- TP3: value TestPoint -> 3v3
- moved D5 28.6 mm to (62.0, 126.5), turned to 180 degrees
- moved R30 27.8 mm to (62.0, 124.5)
- moved TP2 22.5 mm to (84.8, 131.5)
- moved R1 14.9 mm to (62.0, 122.5)
- moved C25 14.9 mm to (80.5, 130.0), turned to 90 degrees
- moved C24 13.8 mm to (67.5, 130.5), turned to 180 degrees
- moved R2 13.1 mm to (62.0, 120.5), turned to 180 degrees
- moved L3 12.8 mm to (75.5, 129.5), turned to 270 degrees
- moved C22 12.3 mm to (73.0, 120.0)
- moved C21 11.7 mm to (68.5, 118.5), turned to 90 degrees
- moved D6 8.74 mm to (76.5, 123.5), turned to 90 degrees
- moved C23 5.34 mm to (74.0, 124.0), turned to 90 degrees
- moved U8 3.36 mm to (68.5, 124.0)
Connections:
- net Net-(C18-Pad1) renamed /3.3V/sw
- net Net-(C23-Pad1) renamed /9V/sw
Routing:
- net Vdrive: track 0.00 -> 18.9 mm
- net GND: track 0.00 -> 6.00 mm, vias 0 -> 5
- net /9V/SNS: track 0.00 -> 5.30 mm
- net Net-(D5-Pad1): track 0.00 -> 3.16 mm
- net Net-(R30-Pad2): track 0.00 -> 2.99 mm
- net Net-(C23-Pad2): track 0.00 -> 2.98 mm
- net Net-(D5-Pad2): track 0.00 -> 2.01 mm
- added copper zone on F.Cu, net +BATT
- added copper zone on F.Cu, net /9V/sw
- added copper zone on B.Cu, net GND
- added copper zone on F.Cu, net GND
- added copper zone on F.Cu, net Vdrive
